Commit message: modify data

File: src/shbat_pkg/urdf/sahabat_robot.urdf.xacro (robot description, xacro)
@@ -1,4 +1,4 @@
 <?xml version = "1.0"?>
-<robot xmlns:xacro="http://www.ros.org/wiki/xacro">
+<robot name="sahabat_robot" xmlns:xacro="http://www.ros.org/wiki/xacro">
 <!--BASE LINK-->
 <link name = "base_link">
@@ -29,4 +29,5 @@
     </visual>
     <collision>
+        <origin xyz = "0.15 0 0.11" />
        <geometry>
             <box size = "0.3 0.35 0.22"/>
@@ -149,5 +150,5 @@
     <collision>
         <geometry>
-            <cylinder radius="0.05" length="0.1"/>
+            <cylinder radius="0.05" length="0.06"/>
         </geometry>
     </collision>
